Commit message: More parts added

File: subwoofer_model/urdf/subwoofer.urdf (robot description, URDF)
Before this commit: robot subwoofer, 5 links, 4 joints
Links:
- added link back_inner_shoulder; visual mesh filename=package://subwoofer_model/meshes/V1.02_Front_Inner_Shoulder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 scale=0.001 0.001 0.001
- added link back_outer_shoulder; visual mesh filename=package://subwoofer_model/meshes/V1.02_Front_Outer_Shoulder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 scale=0.001 0.001 0.001
- added link cover_front; visual mesh filename=package://subwoofer_model/meshes/V1.02_Cover_Nose.stl scale=0.001 0.001 0.001
- added link cover_rear; visual mesh filename=package://subwoofer_model/meshes/V1.02_Cover_Rear_Plain.stl scale=0.001 0.001 0.001
- added link front_inner_shoulder; visual mesh filename=package://subwoofer_model/meshes/V1.02_Front_Inner_Shoulder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 scale=0.001 0.001 0.001
- added link front_outer_shoulder; visual mesh filename=package://subwoofer_model/meshes/V1.02_Front_Outer_Shoulder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 scale=0.001 0.001 0.001
Joints:
- added joint back_inner_shoulder_to_base: type fixed, parent base_link, child back_inner_shoulder, origin xyz=0 -0.063 0.0045
- added joint back_outer_shoulder_to_base: type fixed, parent base_link, child back_outer_shoulder, origin xyz=0 -0.121 0.008
- added joint cover_front_to_base: type fixed, parent base_link, child cover_front, origin xyz=0.0002 0.14 0.004
- added joint cover_rear_to_base: type fixed, parent base_link, child cover_rear, origin xyz=0 -0.145 0.0115
- added joint front_inner_shoulder_to_base: type fixed, parent base_link, child front_inner_shoulder, origin xyz=0 0.064 0.0045
- added joint front_outer_shoulder_to_base: type fixed, parent base_link, child front_outer_shoulder, origin xyz=-0.233 0.117 0.008
- joint cover_bottom_to_base: origin xyz=0 0 -0.035 -> xyz=0 0.005 -0.035
- joint cover_top_to_base: origin xyz=0 0 0.05 -> xyz=0 0.005 0.0455

Commit message: Added servo mesh

File: subwoofer_model/urdf/subwoofer.urdf (robot description, URDF)
Before this commit: robot subwoofer, 11 links, 10 joints
Links:
- added link front_left_hip; visual mesh filename=package://subwoofer_model/meshes/V1.02_Left_Hind_Limb.stl scale=0.001 0.001 0.001
- added link front_left_midlimb; visual mesh filename=package://subwoofer_model/meshes/V1.02_Left_MidLimb.stl scale=0.001 0.001 0.001
- added link front_left_midlimb_cover; visual mesh filename=package://subwoofer_model/meshes/V1.02_Left_MidLimb_Cover.s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 scale=0.001 0.001 0.001
Joints:
- added joint front_left_hip_to_front_shoulder: type revolute, parent front_inner_shoulder, child front_left_hip, origin xyz=-0.039 0.0025 0.0135, axis 0 1 0, limit lower=-0.78 upper=0.78 effort=1000.0 velocity=0.5
- added joint front_left_midlimb_cover_to_midlimb: type fixed, parent front_left_midlimb, child front_left_midlimb_cover, origin xyz=0 0 0
- added joint front_left_midlimb_to_hip: type revolute, parent front_left_hip, child front_left_midlimb, origin xyz=-0.027 0.025 -0.01, axis 1 0 0, limit lower=-0.78 upper=0.78 effort=1000.0 velocity=0.5
