Commit message: Renamed file

File: subwoofer_model/urdf/subwoofer.urdf.xacro (robot description, xacro)
@@ -4,4 +4,9 @@
     <xacro:include filename="$(find subwoofer_model)/urdf/imports/parts.xacro"/>
     <xacro:include filename="$(find subwoofer_model)/urdf/imports/builders.xacro"/>
+    <link name="world"/>
+    <joint name="world_joint" type="fixed">
+        <parent link="world"/>
+        <child link="base_link"/>
+    </joint>
     <xacro:create_body />
     <xacro:create_left_leg
@@ -21,8 +26,3 @@
         name="back_right"
         xyz="${37*scale} ${0*scale} ${7*scale}" />
-    <gazebo>
-        <plugin name="gazebo_ros_control" filename="libgazebo_ros_control.so">
-            <robotNamespace>/</robotNamespace>
-        </plugin>
-    </gazebo>
 </robot>
