Commit message: Fixed file indexing for mesh files

File: subwoofer_model/urdf/imports/parts.xacro (robot description, xacro)
@@ -2,5 +2,5 @@
 <robot xmlns:xacro="http://www.ros.org/wiki/xacro" name="Subwoofer_parts">
     <xacro:include filename="$(find subwoofer_model)/urdf/imports/constants.xacro"/>
-    <xacro:property name="parts_location" value="package://subwoofer_model/meshes"/>
+    <xacro:property name="parts_location" value="file://$(find subwoofer_model)/meshes"/>
     <!-- Servo -->
     <xacro:property name="servo_mesh" value="${parts_location}/Servo.dae" />
