Commit message: Add dynamics properties to joints and update mesh references in URDF and SDF files

File: subwoofer_model/urdf/imports/builders.xacro (robot description, xacro)
@@ -17,8 +17,4 @@
                 </geometry>
             </collision>
-            <inertial>
-                <mass value="${mass}"/>
-                <xacro:default_inertia/>
-            </inertial>
         </link>
     </xacro:macro>
@@ -42,4 +38,5 @@
             <limit effort="1000.0" lower="${lower}" upper="${upper}" velocity="${velocity}"/>
             <origin rpy="${rpy}" xyz="${xyz}"/>
+            <dynamics damping="0.05" friction="0.05"/>
         </joint>
     </xacro:macro>

File: subwoofer_model/urdf/imports/parts.xacro (robot description, xacro)
@@ -99,5 +99,6 @@
     <xacro:property name="right_midlimb_cover_mass" value="0.02"/>
     <!-- Right Wrist -->
-    <xacro:property name="right_wrist_mesh" value="${parts_location}/V1.02_Right_Wrist.stl" />
+    <!--<xacro:property name="right_wrist_mesh" value="${parts_location}/V1.02_Right_Wrist.stl" />-->
+    <xacro:property name="right_wrist_mesh" value="${parts_location}/Right_Wrist.dae" />
     <xacro:property name="right_wrist_xyz" value="${-507*scale} ${235*scale} ${148*scale}"/>
     <xacro:property name="right_wrist_rpy" value="0 1.57075 1.57075"/>

Commit message: Implemented inertial tags for each link in the robot model (still WIP)

File: subwoofer_model/urdf/imports/builders.xacro (robot description, xacro)
@@ -5,4 +5,8 @@
     <xacro:macro name="create_link" params="name mesh rpy xyz mass">
         <link name="${name}">
+            <inertial>
+                <mass value="0.050"/>
+                <inertia ixx="1e-3" ixy="0.0" ixz="0.0" iyy="1e-3" iyz="0.0" izz="1e-3"/>
+            </inertial>
             <visual>
                 <origin rpy="${rpy}" xyz="${xyz}"/>
@@ -19,7 +23,4 @@
         </link>
     </xacro:macro>
-    <xacro:macro name="empty_link" params="name">
-        <link name="${name}"></link>
-    </xacro:macro>
     <!-- Fixed joint -->
     <xacro:macro name="create_fixed_joint" params="parent child rpy xyz">

File: subwoofer_model/urdf/subwoofer.urdf (robot description, URDF)
Before this commit: robot Subwoofer, 39 links, 38 joints
Links:
- added link world
- link back_inner_shoulder: mass 0.018 -> 0.050
- link back_left_hip: mass 0.018 -> 0.050
- link back_left_hip_servo: mass 0.055 -> 0.050
- link back_left_midlimb: mass 0.028 -> 0.050
- link back_left_midlimb_cover: mass 0.02 -> 0.050
- link back_left_midlimb_servo: mass 0.055 -> 0.050
- link back_left_wrist: mass 0.023 -> 0.050
- link back_left_wrist_servo: mass 0.055 -> 0.050
- link back_outer_shoulder: mass 0.034 -> 0.050
- link back_right_hip: mass 0.018 -> 0.050
- link back_right_hip_servo: mass 0.055 -> 0.050
- link back_right_midlimb: mass 0.028 -> 0.050
- link back_right_midlimb_cover: mass 0.02 -> 0.050
- link back_right_midlimb_servo: mass 0.055 -> 0.050
- link back_right_wrist: mass 0.023 -> 0.050; geometry collision mesh filename=package://subwoofer_model/meshes/Right_Wrist.dae scale=0.001 0.001 0.001; visual mesh filename=package://subwoofer_model/meshes/Right_Wrist.dae scale=0.001 0.001 0.001
- link back_right_wrist_servo: mass 0.055 -> 0.050
- link base_link: mass 0.052 -> 0.050
- link bottom_chassis: mass 0.055 -> 0.050
- link front_inner_shoulder: mass 0.035 -> 0.050
- link front_left_hip: mass 0.018 -> 0.050
- link front_left_hip_servo: mass 0.055 -> 0.050
- link front_left_midlimb: mass 0.028 -> 0.050
- link front_left_midlimb_cover: mass 0.02 -> 0.050
- link front_left_midlimb_servo: mass 0.055 -> 0.050
- link front_left_wrist: mass 0.023 -> 0.050
- link front_left_wrist_servo: mass 0.055 -> 0.050
- link front_outer_shoulder: mass 0.017 -> 0.050
- link front_right_hip: mass 0.018 -> 0.050
- link front_right_hip_servo: mass 0.055 -> 0.050
- link front_right_midlimb: mass 0.028 -> 0.050
- link front_right_midlimb_cover: mass 0.02 -> 0.050
- link front_right_midlimb_servo: mass 0.055 -> 0.050
- link front_right_wrist: mass 0.023 -> 0.050; geometry collision mesh filename=package://subwoofer_model/meshes/Right_Wrist.dae scale=0.001 0.001 0.001; visual mesh filename=package://subwoofer_model/meshes/Right_Wrist.dae scale=0.001 0.001 0.001
- link front_right_wrist_servo: mass 0.055 -> 0.050
- link left_chassis: mass 0.011 -> 0.050
- link nose_chassis: mass 0.061 -> 0.050
- link rear_chassis: mass 0.043 -> 0.050
- link right_chassis: mass 0.011 -> 0.050
- link top_chassis: mass 0.06 -> 0.050
Joints:
- added joint world_joint: type fixed, parent world, child base_link
