Commit message: Updated model files to include colours, and changed some rviz default configs

File: subwoofer_model/urdf/imports/builders.xacro (robot description, xacro)
@@ -2,4 +2,5 @@
 <robot xmlns:xacro="http://www.ros.org/wiki/xacro" name="Subwoofer_builders">
     <xacro:include filename="$(find subwoofer_model)/urdf/imports/constants.xacro"/>
+    <xacro:include filename="$(find subwoofer_model)/urdf/imports/materials.xacro"/>
     <!-- Link builder -->
     <xacro:macro name="create_link" params="name mesh rpy xyz mass">
@@ -23,4 +24,25 @@
         </link>
     </xacro:macro>
+    <xacro:macro name="create_link_colour" params="name mesh rpy xyz mass colour">
+        <link name="${name}">
+            <inertial>
+                <mass value="0.050"/>
+                <inertia ixx="1e-3" ixy="0.0" ixz="0.0" iyy="1e-3" iyz="0.0" izz="1e-3"/>
+            </inertial>
+            <visual>
+                <origin rpy="${rpy}" xyz="${xyz}"/>
+                <geometry>
+                    <mesh filename="${mesh}" scale="${scalar}"/>
+                </geometry>
+                <material name="${colour}"/>
+            </visual>
+            <collision>
+                <origin rpy="${rpy}" xyz="${xyz}"/>
+                <geometry>
+                    <mesh filename="${mesh}" scale="${scalar}"/>
+                </geometry>
+            </collision>
+        </link>
+    </xacro:macro>
     <!-- Fixed joint -->
     <xacro:macro name="create_fixed_joint" params="parent child rpy xyz">
@@ -44,6 +66,12 @@
     <!-- Main body builder -->
     <xacro:macro name="create_body">
-        <xacro:create_link
-            name="base_link"
+        <link name="base_link"/>
+        <xacro:create_fixed_joint
+            parent="base_link"
+            child="baseplate"
+            rpy="0 0 0"
+            xyz="0 0 0" />
+        <xacro:create_link
+            name="baseplate"
             mesh="${baseplate_mesh}"
             xyz="${baseplate_xyz}"
@@ -57,5 +85,5 @@
             mass="${front_inner_shoulder_mass}" />
         <xacro:create_fixed_joint
-            parent="base_link"
+            parent="baseplate"
             child="front_inner_shoulder"
             rpy="0 0 0"
@@ -90,5 +118,5 @@
             mass="${back_inner_shoulder_mass}" />
         <xacro:create_fixed_joint
-            parent="base_link"
+            parent="baseplate"
             child="back_inner_shoulder"
             rpy="0 0 0"
@@ -101,5 +129,5 @@
             mass="${chassis_bottom_mass}" />
         <xacro:create_fixed_joint
-            parent="base_link"
+            parent="baseplate"
             child="bottom_chassis"
             rpy="0 0 0"

File: subwoofer_model/urdf/imports/constants.xacro (robot description, xacro)
@@ -6,3 +6,6 @@
         <inertia ixx="1e-3" ixy="0.0" ixz="0.0" iyy="1e-3" iyz="0.0" izz="1e-3"/>
     </xacro:macro>
+    <!-- Colour codes -->
+    <!-- Supernova: 1.0 0.793 0.0 -->
+    <!-- Port Gore: 0.141 0.152 0.328 -->
 </robot>

File: subwoofer_model/urdf/imports/parts.xacro (robot description, xacro)
@@ -4,5 +4,5 @@
     <xacro:property name="parts_location" value="package://subwoofer_model/meshes"/>
     <!-- Servo -->
-    <xacro:property name="servo_mesh" value="${parts_location}/Servo.stl" />
+    <xacro:property name="servo_mesh" value="${parts_location}/Servo.dae" />
     <xacro:property name="servo_xyz" value="${43*scale} ${0*scale} ${-10*scale}"/>
     <xacro:property name="servo_rpy" value="0 3.1415 1.57075"/>
@@ -14,91 +14,90 @@
     <xacro:property name="baseplate_mass" value="0.052"/>
     <!-- Chassis Left -->
-    <xacro:property name="chassis_left_mesh" value="${parts_location}/V1.02_Chassis_Left_Side.stl" />
+    <xacro:property name="chassis_left_mesh" value="${parts_location}/V1.02_Chassis_Left_Side.dae" />
     <xacro:property name="chassis_left_xyz" value="${0*scale} ${0*scale} ${0*scale}"/>
     <xacro:property name="chassis_left_rpy" value="0 0 0"/>
     <xacro:property name="chassis_left_mass" value="0.011"/>
     <!-- Chassis Right -->
-    <xacro:property name="chassis_right_mesh" value="${parts_location}/V1.02_Chassis_Right_Side.stl" />
+    <xacro:property name="chassis_right_mesh" value="${parts_location}/V1.02_Chassis_Right_Side.dae" />
     <xacro:property name="chassis_right_xyz" value="${0*scale} ${0*scale} ${0*scale}"/>
     <xacro:property name="chassis_right_rpy" value="0 0 0"/>
     <xacro:property name="chassis_right_mass" value="0.011"/>
     <!-- Chassis Bottom -->
-    <xacro:property name="chassis_bottom_mesh" value="${parts_location}/V1.02_Cover_Bottom.stl" />
+    <xacro:property name="chassis_bottom_mesh" value="${parts_location}/V1.02_Cover_Bottom.dae" />
     <xacro:property name="chassis_bottom_xyz" value="${1004*scale} ${1015*scale} ${1292*scale}"/>
     <xacro:property name="chassis_bottom_rpy" value="1.57075 0 -1.57075"/>
     <xacro:property name="chassis_bottom_mass" value="0.055"/>
     <!-- Chassis Top -->
-    <xacro:property name="chassis_top_mesh" value="${parts_location}/V1.02_Cover_Top.stl" />
+    <xacro:property name="chassis_top_mesh" value="${parts_location}/V1.02_Cover_Top.dae" />
     <xacro:property name="chassis_top_xyz" value="${1004*scale} ${-1016*scale} ${-1292*scale}"/>
     <xacro:property name="chassis_top_rpy" value="-1.57075 0 1.57075"/>
     <xacro:property name="chassis_top_mass" value="0.06"/>
     <!-- Front shoulder inner -->
-    <xacro:property name="front_inner_shoulder_mesh" value="${parts_location}/V1.02_Front_Inner_Shoulder.stl" />
+    <xacro:property name="front_inner_shoulder_mesh" value="${parts_location}/V1.02_Front_Inner_Shoulder.dae" />
     <xacro:property name="front_inner_shoulder_xyz" value="${-34*scale} ${-2*scale} ${33*scale}"/>
     <xacro:property name="front_inner_shoulder_rpy" value="1.57075 0 3.1415"/>
     <xacro:property name="front_inner_shoulder_mass" value="0.035"/>
     <!-- Front shoulder outer-->
-    <xacro:property name="front_outer_shoulder_mesh" value="${parts_location}/V1.02_Front_Outer_Shoulder.stl" />
+    <xacro:property name="front_outer_shoulder_mesh" value="${parts_location}/V1.02_Front_Outer_Shoulder.dae" />
     <xacro:property name="front_outer_shoulder_xyz" value="${-115.5*scale} ${2*scale} ${467*scale}"/>
     <xacro:property name="front_outer_shoulder_rpy" value="0 3.1415 3.1415"/>
     <xacro:property name="front_outer_shoulder_mass" value="0.017"/>
     <!-- Back shoulder inner -->
-    <xacro:property name="back_inner_shoulder_mesh" value="${parts_location}/V1.02_Rear_Inner_Shoulder.stl" />
+    <xacro:property name="back_inner_shoulder_mesh" value="${parts_location}/V1.02_Rear_Inner_Shoulder.dae" />
     <xacro:property name="back_inner_shoulder_xyz" value="${-116*scale} ${2*scale} ${467*scale}"/>
     <xacro:property name="back_inner_shoulder_rpy" value="3.1415 0 0"/>
     <xacro:property name="back_inner_shoulder_mass" value="0.018"/>
     <!-- Back shoulder outer-->
-    <xacro:property name="back_outer_shoulder_mesh" value="${parts_location}/V1.02_Rear_Outer_Shoulder.stl" />
+    <xacro:property name="back_outer_shoulder_mesh" value="${parts_location}/V1.02_Rear_Outer_Shoulder.dae" />
     <xacro:property name="back_outer_shoulder_xyz" value="${117*scale} ${55*scale} ${-470*scale}"/>
     <xacro:property name="back_outer_shoulder_rpy" value="0 0 3.1415"/>
     <xacro:property name="back_outer_shoulder_mass" value="0.034"/>
     <!-- Chassis Nose -->
-    <xacro:property name="chassis_nose_mesh" value="${parts_location}/V1.02_Cover_Nose.stl" />
+    <xacro:property name="chassis_nose_mesh" value="${parts_location}/V1.02_Cover_Nose.dae" />
     <xacro:property name="chassis_nose_xyz" value="${142*scale} ${355*scale} ${510*scale}"/>
     <xacro:property name="chassis_nose_rpy" value="3.1415 0 1.57075"/>
     <xacro:property name="chassis_nose_mass" value="0.061"/>
     <!-- Chassis Rear -->
-    <xacro:property name="chassis_rear_mesh" value="${parts_location}/V1.02_Cover_Rear_Plain.stl" />
+    <xacro:property name="chassis_rear_mesh" value="${parts_location}/V1.02_Cover_Rear_Plain.dae" />
     <xacro:property name="chassis_rear_xyz" value="${248.7*scale} ${252*scale} ${380*scale}"/>
     <xacro:property name="chassis_rear_rpy" value="0 1.57075 1.57075"/>
     <xacro:property name="chassis_rear_mass" value="0.043"/>
     <!-- Left hind -->
-    <xacro:property name="left_hind_mesh" value="${parts_location}/V1.02_Left_Hind_Limb.stl" />
+    <xacro:property name="left_hind_mesh" value="${parts_location}/V1.02_Left_Hind_Limb.dae" />
     <xacro:property name="left_hind_xyz" value="${3*scale} ${-23*scale} ${-26*scale}"/>
     <xacro:property name="left_hind_rpy" value="0 0 0"/>
     <xacro:property name="left_hind_mass" value="0.018"/>
     <!-- Left midlimb -->
-    <xacro:property name="left_midlimb_mesh" value="${parts_location}/V1.02_Left_MidLimb.stl" />
+    <xacro:property name="left_midlimb_mesh" value="${parts_location}/V1.02_Left_MidLimb.dae" />
     <xacro:property name="left_midlimb_xyz" value="${-48*scale} ${-20*scale} ${825*scale}"/>
     <xacro:property name="left_midlimb_rpy" value="0 3.1415 0"/>
     <xacro:property name="left_midlimb_mass" value="0.028"/>
     <!-- Left midlimb cover -->
-    <xacro:property name="left_midlimb_cover_mesh" value="${parts_location}/V1.02_Left_MidLimb_Cover.stl" />
+    <xacro:property name="left_midlimb_cover_mesh" value="${parts_location}/V1.02_Left_MidLimb_Cover.dae" />
     <xacro:property name="left_midlimb_cover_xyz" value="${256*scale} ${-110*scale} ${926*scale}"/>
     <xacro:property name="left_midlimb_cover_rpy" value="0 3.1415 0"/>
     <xacro:property name="left_midlimb_cover_mass" value="0.02"/>
     <!-- Left Wrist -->
-    <xacro:property name="left_wrist_mesh" value="${parts_location}/V1.02_Left_Wrist.stl" />
+    <xacro:property name="left_wrist_mesh" value="${parts_location}/V1.02_Left_Wrist.dae" />
     <xacro:property name="left_wrist_xyz" value="${507*scale} ${235*scale} ${148*scale}"/>
     <xacro:property name="left_wrist_rpy" value="0 1.57075 -1.57075"/>
     <xacro:property name="left_wrist_mass" value="0.023"/>
     <!-- Right hind -->
-    <xacro:property name="right_hind_mesh" value="${parts_location}/V1.02_Right_Hind_Limb.stl" />
+    <xacro:property name="right_hind_mesh" value="${parts_location}/V1.02_Right_Hind_Limb.dae" />
     <xacro:property name="right_hind_xyz" value="${-120*scale} ${103*scale} ${28.2*scale}"/>
     <xacro:property name="right_hind_rpy" value="3.1415 0 0"/>
     <xacro:property name="right_hind_mass" value="0.018"/>
     <!-- Right midlimb -->
-    <xacro:property name="right_midlimb_mesh" value="${parts_location}/V1.02_Right_MidLimb.stl" />
+    <xacro:property name="right_midlimb_mesh" value="${parts_location}/V1.02_Right_MidLimb.dae" />
     <xacro:property name="right_midlimb_xyz" value="${48*scale} ${-20*scale} ${825*scale}"/>
     <xacro:property name="right_midlimb_rpy" value="0 0 0"/>
     <xacro:property name="right_midlimb_mass" value="0.028"/>
     <!-- Right midlimb cover -->
-    <xacro:property name="right_midlimb_cover_mesh" value="${parts_location}/V1.02_Right_MidLimb_Cover.stl" />
+    <xacro:property name="right_midlimb_cover_mesh" value="${parts_location}/V1.02_Right_MidLimb_Cover.dae" />
     <xacro:property name="right_midlimb_cover_xyz" value="${-256*scale} ${-110*scale} ${926*scale}"/>
     <xacro:property name="right_midlimb_cover_rpy" value="0 0 0"/>
     <xacro:property name="right_midlimb_cover_mass" value="0.02"/>
     <!-- Right Wrist -->
-    <!--<xacro:property name="right_wrist_mesh" value="${parts_location}/V1.02_Right_Wrist.stl" />-->
-    <xacro:property name="right_wrist_mesh" value="${parts_location}/Right_Wrist.dae" />
+    <xacro:property name="right_wrist_mesh" value="${parts_location}/V1.02_Right_Wrist.dae" />
     <xacro:property name="right_wrist_xyz" value="${-507*scale} ${235*scale} ${148*scale}"/>
     <xacro:property name="right_wrist_rpy" value="0 1.57075 1.57075"/>

File: subwoofer_model/urdf/subwoofer.urdf (robot description, URDF)
Before this commit: robot Subwoofer, 40 links, 39 joints
Links:
- added link baseplate, mass 0.050; collision mesh filename=package://subwoofer_model/meshes/V1.02_Chassis_BasePlate_RP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 scale=0.001 0.001 0.001; visual mesh filename=package://subwoofer_model/meshes/V1.02_Chassis_BasePlate_RP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 scale=0.001 0.001 0.001
- link back_left_hip: geometry collision mesh filename=package://subwoofer_model/meshes/V1.02_Left_Hind_Limb.dae scale=0.001 0.001 0.001; visual mesh filename=package://subwoofer_model/meshes/V1.02_Left_Hind_Limb.dae scale=0.001 0.001 0.001
- link back_left_hip_servo: geometry collision mesh filename=package://subwoofer_model/meshes/Servo.dae scale=0.001 0.001 0.001; visual mesh filename=package://subwoofer_model/meshes/Servo.dae scale=0.001 0.001 0.001
- link back_left_midlimb: geometry collision mesh filename=package://subwoofer_model/meshes/V1.02_Left_MidLimb.dae scale=0.001 0.001 0.001; visual mesh filename=package://subwoofer_model/meshes/V1.02_Left_MidLimb.dae scale=0.001 0.001 0.001
- link back_left_midlimb_cover: geometry collision mesh filename=package://subwoofer_model/meshes/V1.02_Left_MidLimb_Cover.d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 scale=0.001 0.001 0.001; visual mesh filename=package://subwoofer_model/meshes/V1.02_Left_MidLimb_Cover.d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 scale=0.001 0.001 0.001
- link back_left_midlimb_servo: geometry collision mesh filename=package://subwoofer_model/meshes/Servo.dae scale=0.001 0.001 0.001; visual mesh filename=package://subwoofer_model/meshes/Servo.dae scale=0.001 0.001 0.001
- link back_left_wrist: geometry collision mesh filename=package://subwoofer_model/meshes/V1.02_Left_Wrist.dae scale=0.001 0.001 0.001; visual mesh filename=package://subwoofer_model/meshes/V1.02_Left_Wrist.dae scale=0.001 0.001 0.001
- link back_left_wrist_servo: geometry collision mesh filename=package://subwoofer_model/meshes/Servo.dae scale=0.001 0.001 0.001; visual mesh filename=package://subwoofer_model/meshes/Servo.dae scale=0.001 0.001 0.001
- link back_right_hip: geometry collision mesh filename=package://subwoofer_model/meshes/V1.02_Right_Hind_Limb.dae scale=0.001 0.001 0.001; visual mesh filename=package://subwoofer_model/meshes/V1.02_Right_Hind_Limb.dae scale=0.001 0.001 0.001
- link back_right_hip_servo: geometry collision mesh filename=package://subwoofer_model/meshes/Servo.dae scale=0.001 0.001 0.001; visual mesh filename=package://subwoofer_model/meshes/Servo.dae scale=0.001 0.001 0.001
- link back_right_midlimb: geometry collision mesh filename=package://subwoofer_model/meshes/V1.02_Right_MidLimb.dae scale=0.001 0.001 0.001; visual mesh filename=package://subwoofer_model/meshes/V1.02_Right_MidLimb.dae scale=0.001 0.001 0.001
- link back_right_midlimb_servo: geometry collision mesh filename=package://subwoofer_model/meshes/Servo.dae scale=0.001 0.001 0.001; visual mesh filename=package://subwoofer_model/meshes/Servo.dae scale=0.001 0.001 0.001
- link back_right_wrist: geometry collision mesh filename=package://subwoofer_model/meshes/V1.02_Right_Wrist.dae scale=0.001 0.001 0.001; visual mesh filename=package://subwoofer_model/meshes/V1.02_Right_Wrist.dae scale=0.001 0.001 0.001
- link back_right_wrist_servo: geometry collision mesh filename=package://subwoofer_model/meshes/Servo.dae scale=0.001 0.001 0.001; visual mesh filename=package://subwoofer_model/meshes/Servo.dae scale=0.001 0.001 0.001
- link base_link: mass 0.050 -> None; geometry 
- link bottom_chassis: geometry collision mesh filename=package://subwoofer_model/meshes/V1.02_Cover_Bottom.dae scale=0.001 0.001 0.001; visual mesh filename=package://subwoofer_model/meshes/V1.02_Cover_Bottom.dae scale=0.001 0.001 0.001
- link front_left_hip: geometry collision mesh filename=package://subwoofer_model/meshes/V1.02_Left_Hind_Limb.dae scale=0.001 0.001 0.001; visual mesh filename=package://subwoofer_model/meshes/V1.02_Left_Hind_Limb.dae scale=0.001 0.001 0.001
- link front_left_hip_servo: geometry collision mesh filename=package://subwoofer_model/meshes/Servo.dae scale=0.001 0.001 0.001; visual mesh filename=package://subwoofer_model/meshes/Servo.dae scale=0.001 0.001 0.001
- link front_left_midlimb: geometry collision mesh filename=package://subwoofer_model/meshes/V1.02_Left_MidLimb.dae scale=0.001 0.001 0.001; visual mesh filename=package://subwoofer_model/meshes/V1.02_Left_MidLimb.dae scale=0.001 0.001 0.001
- link front_left_midlimb_cover: geometry collision mesh filename=package://subwoofer_model/meshes/V1.02_Left_MidLimb_Cover.d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 scale=0.001 0.001 0.001; visual mesh filename=package://subwoofer_model/meshes/V1.02_Left_MidLimb_Cover.d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 scale=0.001 0.001 0.001
- link front_left_midlimb_servo: geometry collision mesh filename=package://subwoofer_model/meshes/Servo.dae scale=0.001 0.001 0.001; visual mesh filename=package://subwoofer_model/meshes/Servo.dae scale=0.001 0.001 0.001
- link front_left_wrist: geometry collision mesh filename=package://subwoofer_model/meshes/V1.02_Left_Wrist.dae scale=0.001 0.001 0.001; visual mesh filename=package://subwoofer_model/meshes/V1.02_Left_Wrist.dae scale=0.001 0.001 0.001
- link front_left_wrist_servo: geometry collision mesh filename=package://subwoofer_model/meshes/Servo.dae scale=0.001 0.001 0.001; visual mesh filename=package://subwoofer_model/meshes/Servo.dae scale=0.001 0.001 0.001
- link front_right_hip: geometry collision mesh filename=package://subwoofer_model/meshes/V1.02_Right_Hind_Limb.dae scale=0.001 0.001 0.001; visual mesh filename=package://subwoofer_model/meshes/V1.02_Right_Hind_Limb.dae scale=0.001 0.001 0.001
- link front_right_hip_servo: geometry collision mesh filename=package://subwoofer_model/meshes/Servo.dae scale=0.001 0.001 0.001; visual mesh filename=package://subwoofer_model/meshes/Servo.dae scale=0.001 0.001 0.001
- link front_right_midlimb: geometry collision mesh filename=package://subwoofer_model/meshes/V1.02_Right_MidLimb.dae scale=0.001 0.001 0.001; visual mesh filename=package://subwoofer_model/meshes/V1.02_Right_MidLimb.dae scale=0.001 0.001 0.001
- link front_right_midlimb_servo: geometry collision mesh filename=package://subwoofer_model/meshes/Servo.dae scale=0.001 0.001 0.001; visual mesh filename=package://subwoofer_model/meshes/Servo.dae scale=0.001 0.001 0.001
- link front_right_wrist: geometry collision mesh filename=package://subwoofer_model/meshes/V1.02_Right_Wrist.dae scale=0.001 0.001 0.001; visual mesh filename=package://subwoofer_model/meshes/V1.02_Right_Wrist.dae scale=0.001 0.001 0.001
- link front_right_wrist_servo: geometry collision mesh filename=package://subwoofer_model/meshes/Servo.dae scale=0.001 0.001 0.001; visual mesh filename=package://subwoofer_model/meshes/Servo.dae scale=0.001 0.001 0.001
- link left_chassis: geometry collision mesh filename=package://subwoofer_model/meshes/V1.02_Chassis_Left_Side.dae scale=0.001 0.001 0.001; visual mesh filename=package://subwoofer_model/meshes/V1.02_Chassis_Left_Side.dae scale=0.001 0.001 0.001
- link nose_chassis: geometry collision mesh filename=package://subwoofer_model/meshes/V1.02_Cover_Nose.dae scale=0.001 0.001 0.001; visual mesh filename=package://subwoofer_model/meshes/V1.02_Cover_Nose.dae scale=0.001 0.001 0.001
- link rear_chassis: geometry collision mesh filename=package://subwoofer_model/meshes/V1.02_Cover_Rear_Plain.dae scale=0.001 0.001 0.001; visual mesh filename=package://subwoofer_model/meshes/V1.02_Cover_Rear_Plain.dae scale=0.001 0.001 0.001
- link right_chassis: geometry collision mesh filename=package://subwoofer_model/meshes/V1.02_Chassis_Right_Side.d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 scale=0.001 0.001 0.001; visual mesh filename=package://subwoofer_model/meshes/V1.02_Chassis_Right_Side.d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 scale=0.001 0.001 0.001
- link top_chassis: geometry collision mesh filename=package://subwoofer_model/meshes/V1.02_Cover_Top.dae scale=0.001 0.001 0.001; visual mesh filename=package://subwoofer_model/meshes/V1.02_Cover_Top.dae scale=0.001 0.001 0.001
Joints:
- removed joint back_inner_shoulder_to_base_link
- removed joint bottom_chassis_to_base_link
- removed joint front_inner_shoulder_to_base_link
- added joint back_inner_shoulder_to_baseplate: type fixed, parent baseplate, child back_inner_shoulder, origin xyz=0.0 -0.066 0.01 rpy=0 0 0
- added joint baseplate_to_base_link: type fixed, parent base_link, child baseplate, origin xyz=0 0 0 rpy=0 0 0
- added joint bottom_chassis_to_baseplate: type fixed, parent baseplate, child bottom_chassis, origin xyz=0.0 0.0 -0.028 rpy=0 0 0
- added joint front_inner_shoulder_to_baseplate: type fixed, parent baseplate, child front_inner_shoulder, origin xyz=0.0 0.065 0.01 rpy=0 0 0
